File: labs_board/labs_board.kicad_pcb (KiCad board)
At the start: 2 copper layers, 260 x 149 mm, 14 parts, among them J1 Conn_Coaxial, J10 Conn_Coaxial, J11 Conn_Coaxial, J12 Conn_Coaxial, J13 Conn_Coaxial, J14 Conn_Coaxial, J2 Conn_Coaxial, J3 Conn_Coaxial, J4 Conn_Coaxial, J5 Conn_Coaxial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

Commit message: second update
Parts:
- moved J10 5.64 mm to (177.0, 150.6)
- moved J9 5.64 mm to (177.0, 28.4)
Other:
- board text added: "50-ohm"
- board text added: "90 Bend"
- board text added: "Bandpass Filter"
- board text added: "Cap Bulge"
- board text added: "EE251 Lab 1"
- board text added: "Experiment Area"
- board text added: "Inductive Notch"
- board text added: "Mitered Bend"
- board text added: "Will Johnson Fengrui Zuo"
Changed lines of the file:
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@@
 			(outputformat 1)
 			(mirror no)
-			(drillshape 1)
+			(drillshape 0)
 			(scaleselection 1)
-			(outputdirectory "")
+			(outputdirectory "job_file/")
 		)
 	)
@@
 	(footprint "Connector_Coaxial:BNC_TEConnectivity_1478204_Vertical"
 		(layer "B.Cu")
-		(at 182.64 28.37 180)
+		(at 177 28.37 180)
 		(descr "BNC female PCB mount 4 pin straight chassis connector http://www.te.com/usa-en/product-1-1478204-0.html")
 		(tags "BNC female PCB mount 4 pin straight chassis connector ")
@@
 	(footprint "Connector_Coaxial:BNC_TEConnectivity_1478204_Vertical"
 		(layer "B.Cu")
-		(at 182.64 150.57 180)
+		(at 177 150.57 180)
 		(descr "BNC female PCB mount 4 pin straight chassis connector http://www.te.com/usa-en/product-1-1478204-0.html")
 		(tags "BNC female PCB mount 4 pin straight chassis connector ")
@@
 		(layer "Edge.Cuts")
 	)
+	(gr_text "Will Johnson\nFengrui Zuo"
+		(at 91 158 90)
+		(layer "F.SilkS")
+		(effects
+			(font
+				(size 4 4)
+				(thickness 0.5)
+			)
+			(justify left bottom)
+		)
+	)
+	(gr_text "Mitered Bend"
+		(at 59 103 90)
+		(layer "F.SilkS")
+		(effects
+			(font
+				(size 4 4)
+				(thickness 0.5)
+			)
+			(justify left bottom)
+		)
+	)
+	(gr_text "Experiment Area"
+		(at 202 112 90)
+		(layer "F.SilkS")
+		(effects
+			(font
+				(size 4 4)
+				(thickness 0.5)
+			)
+			(justify left bottom)
+		)
+	)
+	(gr_text "50-ohm"
+		(at 39 95 90)
+		(layer "F.SilkS")
+		(effects
+			(font
+				(size 4 4)
+				(thickness 0.5)
+			)
+			(justify left bottom)
+		)
+	)
+	(gr_text "90 Bend"
+		(at 89 97 90)
+		(layer "F.SilkS")
+		(effects
+			(font
+				(size 4 4)
+				(thickness 0.5)
+			)
+			(justify left bottom)
+		)
+	)
+	(gr_text "EE251 Lab 1"
+		(at 47 156 90)
+		(layer "F.SilkS")
+		(effects
+			(font
+				(size 4 4)
+				(thickness 0.5)
+			)
+			(justify left bottom)
+		)
+	)
+	(gr_text "Inductive Notch"
+		(at 117 109 90)
+		(layer "F.SilkS")
+		(effects
+			(font
+				(size 4 4)
+				(thickness 0.5)
+			)
+			(justify left bottom)
+		)
+	)
+	(gr_text "Bandpass Filter"
+		(at 168 110 90)
+		(layer "F.SilkS")
+		(effects
+			(font
+				(size 4 4)
+				(thickness 0.5)
+			)
+			(justify left bottom)
+		)
+	)
+	(gr_text "Cap Bulge"
+		(at 136 102 90)
+		(layer "F.SilkS")
+		(effects
+			(font
+				(size 4 4)
+				(thickness 0.5)
+			)
+			(justify left bottom)
+		)
+	)
 	(segment
 		(start 31.8 28.62)
@@
 	)
 	(segment
-		(start 182.58 144.79)
-		(end 182.58 150.77)
+		(start 176.94 144.79)
+		(end 176.94 150.77)
 		(width 1.5)
 		(layer "F.Cu")
@@
 	)
 	(segment
-		(start 182.58 28.39)
-		(end 182.58 35.17)
+		(start 176.94 28.39)
+		(end 176.94 35.17)
 		(width 1.5)
 		(layer "F.Cu")
@@
 	)
 	(segment
-		(start 182.58 35.17)
-		(end 182.58 144.79)
+		(start 176.94 35.17)
+		(end 176.94 144.79)
 		(width 2.71)
 		(layer "F.Cu")

Commit message: 4th updatee
Routing:
- removed copper zone on F.Cu, net /Cap_bulge
Changed lines of the file:
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@@
+	(gr_poly
+		(pts
+			(xy 140 77) (xy 150 77) (xy 150 98) (xy 140 98)
+		)
+		(stroke
+			(width 0.2)
+			(type solid)
+		)
+		(fill solid)
+		(layer "F.Cu")
+		(net 5)
+	)
 	(gr_poly
 		(pts
@@
 	)
 	(zone
-		(net 5)
-		(net_name "/Cap_bulge")
-		(layer "F.Cu")
-		(hatch edge 0.5)
-		(priority 1)
-		(connect_pads
-			(clearance 0.5)
-		)
-		(min_thickness 0.25)
-		(filled_areas_thickness no)
-		(fill yes
-			(thermal_gap 0.5)
-			(thermal_bridge_width 0.5)
-		)
-		(polygon
-			(pts
-				(xy 139.18 79.11) (xy 150.58 79.11) (xy 150.58 94.51) (xy 139.18 94.51)
-			)
-		)
-	)
-	(zone
